File: pcb/attiny1614/AdventSternla.sch (KiCad schematic (older format))
At the start: 13 parts, among them J101 UPDI, J102 NeoPixel Data, J103 Power Out, J104 5V In, J105 GPIO_A, J106 GPIO_B, J107 GPIO_C, U101 ATTINY1614

Commit message: Fixed up the diode foot print
Parts:
- D101: footprint Diodes_SMD:D_SOD-123F -> Diodes_SMD:D_SOD-323
Changed lines of the file:
@@
 F 0 "D101" H 2650 3950 50  0000 C CNN
 F 1 "1N4148WSTR" H 2650 3750 50  0000 C CNN
-F 2 "Diodes_SMD:D_SOD-123F" H 2650 3850 50  0001 C CNN
+F 2 "Diodes_SMD:D_SOD-323" H 2650 3850 50  0001 C CNN
 F 3 "http://www.smc-diodes.com/propdf/1N4148WS%20N0572%20REV.B.pdf" H 2650 3850 50  0001 C CNN
 F 4 "1N4148WSTR" H 2650 3850 60  0001 C CNN "MPN"
