File: pcb/EightChannel/EightChannel.sch (KiCad schematic (older format))
At the start: 11 parts, among them J101 UPDI, J102 5V In, J103 Conn_01x04_Male, J104 Conn_01x07_Male, U101 74LS595, U102 ATTINY1614

Commit message: Finished 8Channel and submitted to Fab
Parts:
- C101, C102, C103: symbol FiveChannel-rescue:C -> EightChannel-rescue:C
- D101: symbol FiveChannel-rescue:D -> EightChannel-rescue:D
- J101: symbol FiveChannel-rescue:Conn_02x03_Odd_Even -> EightChannel-rescue:Conn_02x03_Odd_Even
- J102: symbol FiveChannel-rescue:Jack-DC -> EightChannel-rescue:Jack-DC
- J103: symbol FiveChannel-rescue:Conn_01x04_Male -> EightChannel-rescue:Conn_01x04_Male
- J104: symbol FiveChannel-rescue:Conn_01x07_Male -> EightChannel-rescue:Conn_01x07_Male
- R101: symbol FiveChannel-rescue:R -> EightChannel-rescue:R
- U101: symbol FiveChannel-rescue:74LS596-RESCUE-FiveChannel -> EightChannel-rescue:74LS596-RESCUE-EightChannel
- U102: symbol FiveChannel-rescue:ATTINY1614 -> EightChannel-rescue:ATTINY1614
Changed lines of the file:
@@
 $EndDescr
 $Comp
-L FiveChannel-rescue:ATTINY1614 U102
+L EightChannel-rescue:ATTINY1614 U102
 U 1 1 59EF6A42
 P 5600 4400
@@
 $EndComp
 $Comp
-L FiveChannel-rescue:R R101
+L EightChannel-rescue:R R101
 U 1 1 59EF6A7A
 P 4600 4050
@@
 VDD
 $Comp
-L FiveChannel-rescue:GND #PWR01
+L EightChannel-rescue:GND #PWR01
 U 1 1 59EF6C0B
 P 5600 5550
@@
 Text Label 3800 4300 0    60   ~ 0
 PDI_DATA
-$Comp
-L FiveChannel-rescue:GND #PWR03
+Text Label 1050 1350 0    60   ~ 0
+PDI_DATA
+$Comp
+L EightChannel-rescue:GND #PWR02
+U 1 1 59EF6D08
+P 2250 1750
+F 0 "#PWR02" H 2250 1500 50  0001 C CNN
+F 1 "GND" H 2250 1600 50  0000 C CNN
+F 2 "" H 2250 1750 50  0001 C CNN
+F 3 "" H 2250 1750 50  0001 C CNN
+	1    2250 1750
+	1    0    0    -1
+$EndComp
+Text Label 2450 1350 2    60   ~ 0
+VDD
+$Comp
+L EightChannel-rescue:GND #PWR03
 U 1 1 59EF8502
 P 2550 4900
@@
 	1    0    0    -1
 $EndComp
+$Comp
+L EightChannel-rescue:Conn_02x03_Odd_Even J101
+U 1 1 59EF854F
+P 1700 1450
+F 0 "J101" H 1750 1650 50  0000 C CNN
+F 1 "UPDI" H 1750 1250 50  0000 C CNN
+F 2 "advent_sternla:PRG_TC2030-IDC-NL" H 1700 1450 50  0001 C CNN
+F 3 "" H 1700 1450 50  0001 C CNN
+	1    1700 1450
+	1    0    0    -1
+$EndComp
+NoConn ~ 1500 1450
+NoConn ~ 1500 1550
+NoConn ~ 2000 1450
 Text Label 7750 3850 0    60   ~ 0
 CLK_PIN
@@
 ~ENABLE
 $Comp
-L FiveChannel-rescue:C C102
+L EightChannel-rescue:C C102
 U 1 1 59EF980D
 P 3250 4200
@@
 	1    0    0    -1
 $EndComp
+Text Notes 750  850  0    100  ~ 0
+In System Programming Header - UPDI
 Text Label 2100 3850 0    60   ~ 0
 5V
 $Comp
-L FiveChannel-rescue:Jack-DC J102
+L EightChannel-rescue:Jack-DC J102
 U 1 1 59F100E4
 P 1000 3950
@@
 NeoPixel
 $Comp
-L FiveChannel-rescue:D D101
+L EightChannel-rescue:D D101
 U 1 1 59F5F260
 P 2650 3850
@@
 TODO \nVerify, once more, the Diode i.e. the current rating\nDouble check the connection for the UPDI - is there a need for a \nzero Ohm resistor to deal with any issues?
 $Comp
-L FiveChannel-rescue:74LS596-RESCUE-FiveChannel U101
+L EightChannel-rescue:74LS596-RESCUE-EightChannel U101
 U 1 1 5A60F031
 P 9300 4100
@@
 NoConn ~ 10000 4550
 $Comp
-L FiveChannel-rescue:GND #PWR04
+L EightChannel-rescue:GND #PWR04
 U 1 1 5A60F656
 P 9000 5100
@@
 ~ENABLE
 $Comp
-L FiveChannel-rescue:C C103
+L EightChannel-rescue:C C103
 U 1 1 5A613301
 P 7950 4600
@@
 $EndComp
 $Comp
-L FiveChannel-rescue:GND #PWR05
+L EightChannel-rescue:GND #PWR05
 U 1 1 5A61342B
 P 7950 4900
@@
 $EndComp
 $Comp
-L FiveChannel-rescue:Conn_01x04_Male J103
+L EightChannel-rescue:Conn_01x04_Male J103
 U 1 1 5A64D382
 P 6750 5650
@@
 $EndComp
 $Comp
-L FiveChannel-rescue:Conn_01x07_Male J104
+L EightChannel-rescue:Conn_01x07_Male J104
 U 1 1 5A64D42F
 P 8100 5800
@@
 Connection ~ 4600 4300
 Wire Wire Line
+	1500 1350 1050 1350
+Wire Wire Line
+	2000 1550 2250 1550
+Wire Wire Line
+	2250 1550 2250 1750
+Wire Wire Line
+	2000 1350 2450 1350
+Wire Wire Line
 	1300 3850 1850 3850
 Wire Wire Line
@@
 Wire Wire Line
 	3250 4700 3250 4350
+Wire Notes Line
+	700  900  3000 900
+Wire Notes Line
+	3000 900  3000 2100
+Wire Notes Line
+	3000 2100 700  2100
+Wire Notes Line
+	700  2100 700  900
 Wire Wire Line
 	1500 4700 1850 4700
@@
 DATA_PIN
 $Comp
-L FiveChannel-rescue:C C101
+L EightChannel-rescue:C C101
 U 1 1 5A64D305
 P 1850 4200
@@
 Wire Wire Line
 	1850 4700 2550 4700
-Wire Notes Line
-	700  2100 700  900
-Wire Notes Line
-	3000 2100 700  2100
-Wire Notes Line
-	3000 900  3000 2100
-Wire Notes Line
-	700  900  3000 900
-Wire Wire Line
-	2000 1350 2450 1350
-Wire Wire Line
-	2250 1550 2250 1750
-Wire Wire Line
-	2000 1550 2250 1550
-Wire Wire Line
-	1500 1350 1050 1350
-Text Notes 750  850  0    100  ~ 0
-In System Programming Header - UPDI
-NoConn ~ 2000 1450
-NoConn ~ 1500 1550
-NoConn ~ 1500 1450
-$Comp
-L FiveChannel-rescue:Conn_02x03_Odd_Even J101
-U 1 1 59EF854F
-P 1700 1450
-F 0 "J101" H 1750 1650 50  0000 C CNN
-F 1 "UPDI" H 1750 1250 50  0000 C CNN
-F 2 "advent_sternla:PRG_TC2030-IDC-NL" H 1700 1450 50  0001 C CNN
-F 3 "" H 1700 1450 50  0001 C CNN
-	1    1700 1450
-	1    0    0    -1
-$EndComp
-Text Label 2450 1350 2    60   ~ 0
-VDD
-$Comp
-L FiveChannel-rescue:GND #PWR02
-U 1 1 59EF6D08
-P 2250 1750
-F 0 "#PWR02" H 2250 1500 50  0001 C CNN
-F 1 "GND" H 2250 1600 50  0000 C CNN
-F 2 "" H 2250 1750 50  0001 C CNN
-F 3 "" H 2250 1750 50  0001 C CNN
-	1    2250 1750
-	1    0    0    -1
-$EndComp
-Text Label 1050 1350 0    60   ~ 0
-PDI_DATA
 $EndSCHEMATC
