File: pcb/FiveChannel/Channels.kicad_sch (KiCad schematic)
At the start: 17 parts

Commit message: Hard merge of 5 channel restore (#4)
Co-authored-by: Steve Mayze <smayze@yahoo.com##>
Parts:
- removed J?: NEO STRIPS, symbol Connector:Conn_01x32_Male
- removed R? (x3): 470Ω, Resistors_SMD:R_0805_HandSoldering, symbol FiveChannel-rescue:R
- removed R? (x3): 10kΩ, Resistors_SMD:R_0805_HandSoldering, symbol FiveChannel-rescue:R
- added J201: Conn_01x20_Male, Pin_Headers:Pin_Header_Angled_2x10_Pitch2.54mm, symbol FiveChannel-rescue:Conn_01x20_Male
Connections:
- net 5V_OUT: now also J201.11 (Pin_11), J201.15 (Pin_15), J201.19 (Pin_19), J201.3 (Pin_3), J201.7 (Pin_7)
- net GND: now also J201.10 (Pin_10), J201.12 (Pin_12), J201.14 (Pin_14), J201.16 (Pin_16), J201.18 (Pin_18), J201.2 (Pin_2), J201.20 (Pin_20), J201.4 (Pin_4), J201.6 (Pin_6), J201.8 (Pin_8)
- net NP_DATA_0: now also J201.1 (Pin_1)
- net NP_DATA_1: now also J201.5 (Pin_5)
- net NP_DATA_2: now also J201.9 (Pin_9)
- net NP_DATA_3: now also J201.13 (Pin_13)
- net NP_DATA_4: now also J201.17 (Pin_17)
