File: pcb/FiveChannel/Channels.sch (KiCad schematic (older format))
At the start: 11 parts, among them J201 Conn_01x20_Male

Commit message: Hard merge of 5 channel restore (#4)
Co-authored-by: Steve Mayze <smayze@yahoo.com##>
Parts:
- J201: symbol FiveChannel-rescue:Conn_01x20_Male -> Conn_01x20_Male
- R201, R202, R203, R204, R205, R206, R207, R208, R209, R210: symbol FiveChannel-rescue:R -> R
Changed lines of the file:
@@
-EESchema Schematic File Version 4
-EELAYER 30 0
+EESchema Schematic File Version 2
+LIBS:FiveChannel-rescue
+LIBS:advent_sternla_attiny1614_symbols
+LIBS:SensorBoard
+LIBS:power
+LIBS:device
+LIBS:transistors
+LIBS:conn
+LIBS:linear
+LIBS:regul
+LIBS:74xx
+LIBS:cmos4000
+LIBS:adc-dac
+LIBS:memory
+LIBS:xilinx
+LIBS:microcontrollers
+LIBS:dsp
+LIBS:microchip
+LIBS:analog_switches
+LIBS:motorola
+LIBS:texas
+LIBS:intel
+LIBS:audio
+LIBS:interface
+LIBS:digital-audio
+LIBS:philips
+LIBS:display
+LIBS:cypress
+LIBS:siliconi
+LIBS:opto
+LIBS:atmel
+LIBS:contrib
+LIBS:valves
+EELAYER 25 0
 EELAYER END
 $Descr A4 11693 8268
@@
 $EndDescr
 $Comp
-L FiveChannel-rescue:R R201
+L R R201
 U 1 1 5A6109CB
 P 2800 1750
@@
 NP_DATA_0
 $Comp
-L FiveChannel-rescue:R R202
+L R R202
 U 1 1 5A6109F1
 P 2250 2050
@@
 $EndComp
 $Comp
-L FiveChannel-rescue:GND #PWR06
+L GND #PWR06
 U 1 1 5A6109FB
 P 2250 2450
@@
 5V_OUT
 $Comp
-L FiveChannel-rescue:R R203
+L R R203
 U 1 1 5A610BFB
 P 2800 2850
@@
 NP_DATA_1
 $Comp
-L FiveChannel-rescue:R R204
+L R R204
 U 1 1 5A610C1C
 P 2250 3150
@@
 $EndComp
 $Comp
-L FiveChannel-rescue:GND #PWR07
+L GND #PWR07
 U 1 1 5A610C25
 P 2250 3550
@@
 CHANNEL_1
 $Comp
-L FiveChannel-rescue:R R205
+L R R205
 U 1 1 5A610CEF
 P 2800 3900
@@
 NP_DATA_2
 $Comp
-L FiveChannel-rescue:R R206
+L R R206
 U 1 1 5A610D10
 P 2250 4200
@@
 $EndComp
 $Comp
-L FiveChannel-rescue:GND #PWR08
+L GND #PWR08
 U 1 1 5A610D19
 P 2250 4600
@@
 CHANNEL_2
 $Comp
-L FiveChannel-rescue:R R207
+L R R207
 U 1 1 5A610DC7
 P 2800 4950
@@
 NP_DATA_3
 $Comp
-L FiveChannel-rescue:R R208
+L R R208
 U 1 1 5A610DE8
 P 2250 5250
@@
 $EndComp
 $Comp
-L FiveChannel-rescue:GND #PWR09
+L GND #PWR09
 U 1 1 5A610DF1
 P 2250 5650
@@
 CHANNEL_3
 $Comp
-L FiveChannel-rescue:R R209
+L R R209
 U 1 1 5A61102D
 P 2800 6050
@@
 NP_DATA_4
 $Comp
-L FiveChannel-rescue:R R210
+L R R210
 U 1 1 5A61104E
 P 2250 6350
@@
 $EndComp
 $Comp
-L FiveChannel-rescue:GND #PWR010
+L GND #PWR010
 U 1 1 5A611057
 P 2250 6750
@@
 GND
 $Comp
-L FiveChannel-rescue:Conn_01x20_Male J201
+L Conn_01x20_Male J201
 U 1 1 5A64B1D0
 P 5200 2600
