File: pcb/FiveChannel/FiveChannel.kicad_sch (KiCad schematic)
At the start: 11 parts, among them J101 UPDI, J102 5V In, J103 Conn_01x04_Male, J104 Conn_01x07_Male, U101 74LS595, U102 ATTINY1614

Commit message: Hard merge of 5 channel restore (#4)
Co-authored-by: Steve Mayze <smayze@yahoo.com##>
Parts:
- U102: symbol FiveChannel-rescue:ATTINY1614 -> advent_sternla_attiny1614_symbols:ATTINY1614
Connections:
- net CHANNEL_5: no longer names the net of U101.5 (QF)
- net CHANNEL_6: no longer names the net of U101.6 (QG)
- net CHANNEL_7: no longer names the net of U101.7 (QH)
- no-connect marks 5 -> 8
Other:
- sheet Channels ports: added none; removed CHANNEL_5, CHANNEL_6, CHANNEL_7
