File: pcb/FiveChannel/FiveChannel.sch (KiCad schematic (older format))
At the start: 11 parts, among them J101 UPDI, J102 5V In, J103 Conn_01x04_Male, J104 Conn_01x07_Male, U101 74LS595, U102 ATTINY1614

Commit message: Hard merge of 5 channel restore (#4)
Co-authored-by: Steve Mayze <smayze@yahoo.com##>
Parts:
- C101, C102, C103: symbol FiveChannel-rescue:C -> C
- D101: symbol FiveChannel-rescue:D -> D
- J101: symbol FiveChannel-rescue:Conn_02x03_Odd_Even -> Conn_02x03_Odd_Even
- J102: symbol FiveChannel-rescue:Jack-DC -> Jack-DC
- J103: symbol FiveChannel-rescue:Conn_01x04_Male -> Conn_01x04_Male
- J104: symbol FiveChannel-rescue:Conn_01x07_Male -> Conn_01x07_Male
- R101: symbol FiveChannel-rescue:R -> R
- U101: symbol FiveChannel-rescue:74LS596-RESCUE-FiveChannel -> 74LS596-RESCUE-FiveChannel
- U102: symbol FiveChannel-rescue:ATTINY1614 -> ATTINY1614
Changed lines of the file:
@@
-EESchema Schematic File Version 4
-EELAYER 30 0
+EESchema Schematic File Version 2
+LIBS:FiveChannel-rescue
+LIBS:advent_sternla_attiny1614_symbols
+LIBS:SensorBoard
+LIBS:power
+LIBS:device
+LIBS:transistors
+LIBS:conn
+LIBS:linear
+LIBS:regul
+LIBS:74xx
+LIBS:cmos4000
+LIBS:adc-dac
+LIBS:memory
+LIBS:xilinx
+LIBS:microcontrollers
+LIBS:dsp
+LIBS:microchip
+LIBS:analog_switches
+LIBS:motorola
+LIBS:texas
+LIBS:intel
+LIBS:audio
+LIBS:interface
+LIBS:digital-audio
+LIBS:philips
+LIBS:display
+LIBS:cypress
+LIBS:siliconi
+LIBS:opto
+LIBS:atmel
+LIBS:contrib
+LIBS:valves
+EELAYER 25 0
 EELAYER END
 $Descr A4 11693 8268
@@
 $EndDescr
 $Comp
-L FiveChannel-rescue:ATTINY1614 U102
+L ATTINY1614 U102
 U 1 1 59EF6A42
 P 5600 4400
@@
 $EndComp
 $Comp
-L FiveChannel-rescue:R R101
+L R R101
 U 1 1 59EF6A7A
 P 4600 4050
@@
 VDD
 $Comp
-L FiveChannel-rescue:GND #PWR01
+L GND #PWR01
 U 1 1 59EF6C0B
 P 5600 5550
@@
 PDI_DATA
 $Comp
-L FiveChannel-rescue:GND #PWR02
+L GND #PWR02
 U 1 1 59EF6D08
 P 2250 1750
@@
 VDD
 $Comp
-L FiveChannel-rescue:GND #PWR03
+L GND #PWR03
 U 1 1 59EF8502
 P 2550 4900
@@
 $EndComp
 $Comp
-L FiveChannel-rescue:Conn_02x03_Odd_Even J101
+L Conn_02x03_Odd_Even J101
 U 1 1 59EF854F
 P 1700 1450
@@
 ~ENABLE
 $Comp
-L FiveChannel-rescue:C C102
+L C C102
 U 1 1 59EF980D
 P 3250 4200
@@
 5V
 $Comp
-L FiveChannel-rescue:Jack-DC J102
+L Jack-DC J102
 U 1 1 59F100E4
 P 1000 3950
@@
 NeoPixel
 $Comp
-L FiveChannel-rescue:D D101
+L D D101
 U 1 1 59F5F260
 P 2650 3850
@@
 TODO \nVerify, once more, the Diode i.e. the current rating\nDouble check the connection for the UPDI - is there a need for a \nzero Ohm resistor to deal with any issues?
 $Comp
-L FiveChannel-rescue:74LS596-RESCUE-FiveChannel U101
+L 74LS596-RESCUE-FiveChannel U101
 U 1 1 5A60F031
 P 9300 4100
@@
 NoConn ~ 10000 4550
 $Comp
-L FiveChannel-rescue:GND #PWR04
+L GND #PWR04
 U 1 1 5A60F656
 P 9000 5100
@@
 ~ENABLE
 $Comp
-L FiveChannel-rescue:C C103
+L C C103
 U 1 1 5A613301
 P 7950 4600
@@
 $EndComp
 $Comp
-L FiveChannel-rescue:GND #PWR05
+L GND #PWR05
 U 1 1 5A61342B
 P 7950 4900
@@
 $EndComp
 $Comp
-L FiveChannel-rescue:Conn_01x04_Male J103
+L Conn_01x04_Male J103
 U 1 1 5A64D382
 P 6750 5650
@@
 $EndComp
 $Comp
-L FiveChannel-rescue:Conn_01x07_Male J104
+L Conn_01x07_Male J104
 U 1 1 5A64D42F
 P 8100 5800
@@
 $EndComp
 Wire Wire Line
-	3800 4300 4600 4300
+	3800 4300 4800 4300
 Wire Wire Line
 	4600 4300 4600 4200
@@
 	2000 1350 2450 1350
 Wire Wire Line
-	1300 3850 1850 3850
+	1300 3850 2500 3850
 Wire Wire Line
 	3250 3850 3250 4050
@@
 	700  2100 700  900
 Wire Wire Line
-	1500 4700 1850 4700
+	1500 4700 3250 4700
 Wire Wire Line
 	2550 4700 2550 4900
@@
 Connection ~ 2000 3850
 Wire Wire Line
-	2800 3850 3250 3850
+	2800 3850 4800 3850
 Connection ~ 3250 3850
 Wire Wire Line
@@
 	8200 3950 8600 3950
 Wire Wire Line
-	6450 4150 7950 4150
+	6450 4150 8600 4150
 Wire Wire Line
 	6450 4300 7150 4300
@@
 DATA_PIN
 $Comp
-L FiveChannel-rescue:C C101
+L C C101
 U 1 1 5A64D305
 P 1850 4200
@@
 Text Label 4650 2750 0    60   ~ 0
 5V_OUT
-Wire Wire Line
-	4600 4300 4800 4300
-Wire Wire Line
-	2550 4700 3250 4700
-Wire Wire Line
-	2000 3850 2500 3850
-Wire Wire Line
-	3250 3850 4600 3850
-Wire Wire Line
-	4600 3850 4800 3850
-Wire Wire Line
-	7950 4150 8600 4150
-Wire Wire Line
-	1850 3850 2000 3850
-Wire Wire Line
-	1850 4700 2550 4700
 $EndSCHEMATC
